Commit message: 新增 3D 激光仿真车与 RViz 控制面板，修复代价地图显示
- pnc_nav_sim：万向轮改为前后两个（参考 MoveXBot），
  新增 Velodyne VLP-16 风格 3D 激光版同款车（16线/360°，
  diff_drive_3d + bridge_3d + gz_3d_lidar launch），
  gz_playground 参数化支持 2D/3D 切换
- pnc_nav_rviz：新增 RViz 控制面板插件（移动控制 / 保存地图 /
  AMCL 重定位 / 待扩展按键）
- pnc_nav_core：nav_server 新增 /costmap 代价地图发布（RViz 可视化膨胀层）
- pnc_nav_planners：DWA headingCost 改进（目标方向角驱动 +
  近目标切换 goal yaw 转正），附带调试输出
- AMCL 参数调优（粒子数 5000、更新频率提高）、初始位姿对齐
- Dockerfile 增加中文字体（修复 RViz 中文乱码）

File: src/pnc_nav_sim/urdf/diff_drive_3d.urdf.xacro (robot description, xacro)
@@ -142,10 +142,10 @@
     <axis xyz="1 1 1"/>
   </joint>
-  <!-- LiDAR: gpu_lidar (Harmonic), mounted on top of base_link -->
-  <link name="laser">
-    <visual>
-      <origin xyz="0 0 0" rpy="0 0 0"/>
-      <geometry>
-        <cylinder radius="0.04" length="0.05"/>
+  <!-- 3D LiDAR: Velodyne VLP-16 风格（16 线），车顶安装 -->
+  <link name="velodyne">
+    <visual>
+      <origin xyz="0 0 0" rpy="0 0 0"/>
+      <geometry>
+        <cylinder radius="0.05" length="0.08"/>
       </geometry>
       <material name="dark">
@@ -156,16 +156,16 @@
       <origin xyz="0 0 0" rpy="0 0 0"/>
       <geometry>
-        <cylinder radius="0.04" length="0.05"/>
-      </geometry>
-    </collision>
-    <inertial>
-      <mass value="0.1"/>
-      <inertia ixx="0.0001" ixy="0.0" ixz="0.0" iyy="0.0001" iyz="0.0" izz="0.0001"/>
-    </inertial>
-  </link>
-  <joint name="laser_joint" type="fixed">
-    <parent link="base_link"/>
-    <child link="laser"/>
-    <origin xyz="0 0 0.25" rpy="0 0 0"/>
+        <cylinder radius="0.05" length="0.08"/>
+      </geometry>
+    </collision>
+    <inertial>
+      <mass value="0.6"/>
+      <inertia ixx="0.0004" ixy="0.0" ixz="0.0" iyy="0.0004" iyz="0.0" izz="0.0005"/>
+    </inertial>
+  </link>
+  <joint name="velodyne_joint" type="fixed">
+    <parent link="base_link"/>
+    <child link="velodyne"/>
+    <origin xyz="0 0 0.30" rpy="0 0 0"/>
   </joint>
   <gazebo reference="base_link">
@@ -243,24 +243,30 @@
     </plugin>
   </gazebo>
-  <!-- LiDAR sensor: gpu_lidar (same style as movexbot laser.xacro) -->
-  <gazebo reference="laser">
-    <sensor type="gpu_lidar" name="laser_sensor">
+  <!-- Velodyne VLP-16 风格：16 线，水平 360°，垂直 ±15°，10Hz -->
+  <gazebo reference="velodyne">
+    <sensor type="gpu_lidar" name="velodyne_sensor">
       <pose>0 0 0 0 0 0</pose>
       <visualize>false</visualize>
-      <update_rate>100</update_rate>
-      <topic>nav_scan</topic>
-      <gz_frame_id>laser</gz_frame_id>
+      <update_rate>10</update_rate>
+      <topic>/points</topic>
+      <gz_frame_id>velodyne</gz_frame_id>
       <lidar>
         <scan>
           <horizontal>
-            <samples>720</samples>
+            <samples>1800</samples>
             <resolution>1</resolution>
-            <min_angle>-2.09</min_angle>
-            <max_angle>2.09</max_angle>
+            <min_angle>-3.14159265</min_angle>
+            <max_angle>3.14159265</max_angle>
           </horizontal>
+          <vertical>
+            <samples>16</samples>
+            <resolution>1</resolution>
+            <min_angle>-0.261799</min_angle>
+            <max_angle>0.261799</max_angle>
+          </vertical>
         </scan>
         <range>
-          <min>0.10</min>
-          <max>40.0</max>
+          <min>0.5</min>
+          <max>100.0</max>
           <resolution>0.01</resolution>
         </range>
